File: Boat_PCB/Boat_PCB_V3_1/Boat_PCB_V3_1.kicad_sch (KiCad schematic)
At the start: 75 parts, among them J1 XT60 10S PACK IN, J10 Qwiic spare, J11 Hull leak L, J12 Hull leak R, J13 Winch ESC, J14 Winch home switch, J15 Drive L ESC, J16 Drive R ESC, J17 2nd Pico, J2 Raspberry Pi 5 GPIO, J3 CAN A, J4 CAN B, J5 Pod tether 15V, J6 GPS M10 + compass, J7 RC receiver, J8 SHT41 module GY-SHT41-D, J9 Qwiic TMP119 water, Q1 IRF9540N, Q2 BSS138, SW1 PICO RESET, U1 Pololu D36V50F5 5V 5.5A, U2 Pololu D36V6F15 15V 600mA, U3 Raspberry Pi Pico 2, U4 TJA1051T/3, U5 THVD2410

Commit message: feat(pcb): V3 carrier rev E: two Pico 2s, Pi link on the header
Rev E replaces the Teensy 4.1 with two Raspberry Pi Pico 2s, one job each,
after V3.1 tried one Pico: Pico A (U1) runs control (CAN on can2040, SBUS,
winch, stepper, LED, leak sensing, 12S ADC) and Pico B (U14) the sensors
(I2C mux, GPS, pod RS-485), joined by a UART link. Both are socketed under
the carrier, take VSYS from +5V through D10/D11 and have reset buttons
SW1/SW2. R36/R62 drop to 4.7k for RP2350 erratum E9.

The Pi talks to Pico A over its GPIO header instead of USB, so its USB
ports stay free for cameras and the modem: Pi UART0 (GPIO14/15) runs to
Pico A GP17/GP16 through 1k series resistors (R66/R67), so neither end can
back-power the other, and GPIO23/24 reset Pico A/B through BSS138s (Q3/Q4)
across SW1/SW2, held off by 100k pull-downs (R64/R65). The Picos' USB stays
usable: VBUS isn't wired on the carrier.

C25 (A4988 VMOT bulk) goes from 100 uF to 470 uF 35 V, so C1, C2, C25 and
C26 all take the Rubycon caps already on hand (listed in the parts doc).

Library: RaspberryPi_Pico pin 3 (GND) is power_in now, since two Picos on
one GND net were a power-output conflict; the V3.1 schematic gets a GND
PWR_FLAG to match.

Boat_PCB_V3, rev D -> rev E: 126 -> 137 footprints, 5356 -> 4198 mm of
track, 142 -> 118 vias. DRC 0 -> 0, unconnected 0 -> 0, schematic parity
0 -> 0, ERC 0 -> 0. Boat_PCB_V3_1 and Pod_PCB_V3: DRC, parity and ERC stay
at 0.

Docs: CLAUDE.md pin maps and hardware facts, README, design brief, V3 docs
index, V3.1 doc, session context, parts doc and lib README; this week's
update bullet.

Co-Authored-By: Claude Opus 5.5 <noreply@anthropic.com>
Changed lines of the file:
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@@
+		)
+	)
+	(symbol
+		(lib_id "power:PWR_FLAG")
+		(at 45.72 43.18 0)
+		(unit 1)
+		(body_style 1)
+		(exclude_from_sim no)
+		(in_bom no)
+		(on_board no)
+		(in_pos_files yes)
+		(dnp no)
+		(property "Reference" "#FLG03"
+			(at 45.72 38.10 0)
+			(hide yes)
+			(do_not_autoplace no)
+			(effects
+				(font
+					(size 1.27 1.27)
+				)
+			)
+		)
+		(property "Value" "PWR_FLAG"
+			(at 45.72 39.37 0)
+			(do_not_autoplace no)
+			(effects
+				(font
+					(size 1.27 1.27)
+				)
+			)
+		)
+		(property "Footprint" ""
+			(at 45.72 43.18 0)
+			(hide yes)
+			(do_not_autoplace no)
+			(effects
+				(font
+					(size 1.27 1.27)
+				)
+			)
+		)
+		(property "Datasheet" ""
+			(at 45.72 43.18 0)
+			(hide yes)
+			(do_not_autoplace no)
+			(effects
+				(font
+					(size 1.27 1.27)
+				)
+			)
+		)
+		(property "Description" ""
+			(at 45.72 43.18 0)
+			(hide yes)
+			(do_not_autoplace no)
+			(effects
+				(font
+					(size 1.27 1.27)
+				)
+			)
+		)
+		(pin "1"
+		)
+		(instances
+			(project "Boat_PCB_V3_1"
+				(path "/f04ccb01-50e1-5ad8-9dcc-9a7a44265a94"
+					(reference "#FLG03")
+					(unit 1)
+				)
+			)
+		)
+	)
+	(symbol
+		(lib_id "power:GND")
+		(at 45.72 43.18 0)
+		(unit 1)
+		(body_style 1)
+		(exclude_from_sim no)
+		(in_bom no)
+		(on_board no)
+		(in_pos_files yes)
+		(dnp no)
+		(property "Reference" "#PWR086"
+			(at 45.72 43.18 0)
+			(hide yes)
+			(do_not_autoplace no)
+			(effects
+				(font
+					(size 1.27 1.27)
+				)
+			)
+		)
+		(property "Value" "GND"
+			(at 45.72 47.38 0)
+			(do_not_autoplace no)
+			(effects
+				(font
+					(size 1.27 1.27)
+				)
+			)
+		)
+		(property "Footprint" ""
+			(at 45.72 43.18 0)
+			(hide yes)
+			(do_not_autoplace no)
+			(effects
+				(font
+					(size 1.27 1.27)
+				)
+			)
+		)
+		(property "Datasheet" ""
+			(at 45.72 43.18 0)
+			(hide yes)
+			(do_not_autoplace no)
+			(effects
+				(font
+					(size 1.27 1.27)
+				)
+			)
+		)
+		(property "Description" ""
+			(at 45.72 43.18 0)
+			(hide yes)
+			(do_not_autoplace no)
+			(effects
+				(font
+					(size 1.27 1.27)
+				)
+			)
+		)
+		(pin "1"
+		)
+		(instances
+			(project "Boat_PCB_V3_1"
+				(path "/f04ccb01-50e1-5ad8-9dcc-9a7a44265a94"
+					(reference "#PWR086")
+					(unit 1)
+				)
+			)
 		)
 	)
