File: Boat_PCB/Boat_PCB_V3_1/Boat_PCB_V3_1.kicad_pcb (KiCad board)
At the start: 2 copper layers, 98 x 67 mm, 75 parts, among them J1 XT60 10S PACK IN, J10 Qwiic spare, J11 Hull leak L, J12 Hull leak R, J13 Winch ESC, J14 Winch home switch, J15 Drive L ESC, J16 Drive R ESC, J17 2nd Pico, J2 Raspberry Pi 5 GPIO, J3 CAN A, J4 CAN B, J5 Pod tether 15V, J6 GPS M10 + compass, J7 RC receiver, J8 SHT41 module GY-SHT41-D, J9 Qwiic TMP119 water, Q1 IRF9540N, Q2 BSS138, SW1 PICO RESET, U1 Pololu D36V50F5 5V 5.5A, U2 Pololu D36V6F15 15V 600mA, U3 Raspberry Pi Pico 2, U4 TJA1051T/3, U5 THVD2410

Commit message: chore(pcb): V3.1 order-number marker for PCBWay
The V3.1 starter carrier is being ordered from PCBWay, so the back-silk
order-number marker under the Pico changes from JLCPCB's "JLCJLCJLCJLC" to
PCBWay's "WayWayWay" (same spot, size and angle). Pick "Specify a location"
for the product number at checkout and PCBWay prints it there. Silkscreen
only: the back silkscreen gerber is the only one that changes.

Boat_PCB_V3_1 (rev A): 98.1 x 67.1 mm, 75 footprints, unchanged.
DRC 0 -> 0, unconnected 0 -> 0, schematic parity 0 -> 0, ERC 0 -> 0.

Co-Authored-By: Claude Opus 5.5 <noreply@anthropic.com>
Other:
- board text added: "WayWayWay"
- board text removed: "JLCJLCJLCJLC"
Changed lines of the file:
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@@
 		)
 	)
-	(gr_text "JLCJLCJLCJLC"
+	(gr_text "WayWayWay"
 		(at 127.03 61.61 90)
 		(layer "B.SilkS")
