File: Boat_PCB/Boat_PCB_V3/Boat_PCB_V3.kicad_pcb (KiCad board)
At the start: 4 copper layers, 130.6 x 101.5 mm, 126 parts, among them J1 GPS M10-25Q, J10 Winch ESC, J11 12S HV tap (JST-VH), J12 Raspberry Pi 5 GPIO, J13 XT60 M18 ELECTRONICS, J14 XT60 M18 WINCH, J16 XT60-F WINCH ESC OUT (female), J2 Pod tether, J3 CAN stub to VESCs, J4 SHT45 external, J5 Radar stepper motor, J6 Status LED, J7 SBUS RC receiver, J8 Hull leak left, J9 Hull leak right, Q1 IPP120P04P4L-03, Q2 BSS138, U1 Teensy4.1, U10 INA228 electronics, U11 INA228 winch, U12 74AHCT1G125, U13 THVD2410, U2 TCA9548A I2C mux, U3 TJA1051T/3 CAN xcvr, U4 BNO085, U5 ADXL375, U6 BMP390 breakout, U7 BH1750FVI-TR, U8 SHT45 internal, Y1 32.768kHz CL=12.5pF 50ppm

Commit message: feat(pcb): V3 carrier rev E: two Pico 2s, Pi link on the header
Rev E replaces the Teensy 4.1 with two Raspberry Pi Pico 2s, one job each,
after V3.1 tried one Pico: Pico A (U1) runs control (CAN on can2040, SBUS,
winch, stepper, LED, leak sensing, 12S ADC) and Pico B (U14) the sensors
(I2C mux, GPS, pod RS-485), joined by a UART link. Both are socketed under
the carrier, take VSYS from +5V through D10/D11 and have reset buttons
SW1/SW2. R36/R62 drop to 4.7k for RP2350 erratum E9.

The Pi talks to Pico A over its GPIO header instead of USB, so its USB
ports stay free for cameras and the modem: Pi UART0 (GPIO14/15) runs to
Pico A GP17/GP16 through 1k series resistors (R66/R67), so neither end can
back-power the other, and GPIO23/24 reset Pico A/B through BSS138s (Q3/Q4)
across SW1/SW2, held off by 100k pull-downs (R64/R65). The Picos' USB stays
usable: VBUS isn't wired on the carrier.

C25 (A4988 VMOT bulk) goes from 100 uF to 470 uF 35 V, so C1, C2, C25 and
C26 all take the Rubycon caps already on hand (listed in the parts doc).

Library: RaspberryPi_Pico pin 3 (GND) is power_in now, since two Picos on
one GND net were a power-output conflict; the V3.1 schematic gets a GND
PWR_FLAG to match.

Boat_PCB_V3, rev D -> rev E: 126 -> 137 footprints, 5356 -> 4198 mm of
track, 142 -> 118 vias. DRC 0 -> 0, unconnected 0 -> 0, schematic parity
0 -> 0, ERC 0 -> 0. Boat_PCB_V3_1 and Pod_PCB_V3: DRC, parity and ERC stay
at 0.

Docs: CLAUDE.md pin maps and hardware facts, README, design brief, V3 docs
index, V3.1 doc, session context, parts doc and lib README; this week's
update bullet.

Co-Authored-By: Claude Opus 5.5 <noreply@anthropic.com>
Parts:
- added D10: B5819W, dreams_v3:D_SOD-123, F.Cu at (95.2, 87.5)
- added D11: B5819W, dreams_v3:D_SOD-123, F.Cu at (118.0, 85.6)
- added Q3: BSS138, dreams_v3:SOT-23, F.Cu at (118.6, 21.6)
- added Q4: BSS138, dreams_v3:SOT-23, F.Cu at (118.6, 25.4)
- added R64: 100k 1%, dreams_v3:R_Axial_DIN0207_L6.3mm_D2.5mm_P10.16mm_Horizontal, F.Cu at (114.2, 21.6)
- added R65: 100k 1%, dreams_v3:R_Axial_DIN0207_L6.3mm_D2.5mm_P10.16mm_Horizontal, F.Cu at (114.2, 25.4)
- added R66: 1k 1%, dreams_v3:R_Axial_DIN0207_L6.3mm_D2.5mm_P2.54mm_Vertical, F.Cu at (82.0, 31.6)
- added R67: 1k 1%, dreams_v3:R_Axial_DIN0207_L6.3mm_D2.5mm_P2.54mm_Vertical, F.Cu at (82.0, 35.4)
- added SW1: PICO A RESET, dreams_v3:SW_PUSH_6mm, B.Cu at (129.2, 91.2)
- added SW2: PICO B RESET, dreams_v3:SW_PUSH_6mm, B.Cu at (129.2, 81.2)
- added U14: Raspberry Pi Pico 2, dreams_v3:RaspberryPi_Pico_Socketed_THT, B.Cu at (104.0, 91.0)
- C25: value 100uF 35V -> 470uF 35V
- R36, R62: value 10k 1% -> 4.7k 1%
- U1: value Teensy4.1 -> Raspberry Pi Pico 2; footprint dreams_v3:Teensy41 -> dreams_v3:RaspberryPi_Pico_Socketed_THT
- moved R42 69.5 mm to (94.9, 84.8), turned to 180 degrees
- moved U1 51.7 mm to (82.3, 91.0), turned to 0 degrees
- moved R40 41.2 mm to (94.9, 81.4), turned to 180 degrees
- moved R25 37.4 mm to (117.8, 78.7), turned to 180 degrees
- moved R26 37.4 mm to (117.8, 82.1), turned to 180 degrees
- moved R29 37.4 mm to (117.8, 71.9), turned to 180 degrees
- moved R27 36.4 mm to (117.8, 65.1), turned to 180 degrees
- moved R28 36.4 mm to (117.8, 68.5), turned to 180 degrees
- moved R30 35.8 mm to (117.8, 75.3), turned to 180 degrees
- moved R38 34.1 mm to (114.2, 33.5), turned to 180 degrees
- moved C4 31.3 mm to (97.6, 68.1)
- moved R17 28.2 mm to (117.8, 58.3), turned to 180 degrees
- moved R9 26.7 mm to (117.8, 51.5), turned to 180 degrees
- moved R18 23.4 mm to (117.8, 61.7), turned to 180 degrees
- moved TP5 23.3 mm to (105.5, 38.0)
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Connections:
- J12 pad 10: unconnected-(J12-GPIO15_RXD-Pad10) -> /PI_RX
- J12 pad 16: unconnected-(J12-GPIO23-Pad16) -> /PI_RST_A
- J12 pad 18: unconnected-(J12-GPIO24-Pad18) -> /PI_RST_B
- J12 pad 8: unconnected-(J12-GPIO14_TXD-Pad8) -> /PI_TX
- U1 pad 1: GND -> /WINCH_PWM
- U1 pad 10: /STEP_EN -> /STEP_MS1
- U1 pad 11: /MUX_RST -> /STEP_EN
- U1 pad 12: /IMU_RST -> /WINCH_KILL
- U1 pad 13: /IMU_INT -> GND
- U1 pad 14: /INA_ALERT -> /LED_DIN
- U1 pad 15: +3V3 -> /PWR_GOOD
- U1 pad 16: /BMP_INT -> unconnected-(U1-GPIO12-Pad16)
- U1 pad 17: /STEP_MS1 -> unconnected-(U1-GPIO13-Pad17)
- U1 pad 18: /STEP_MS2 -> GND
- U1 pad 19: /STEP_MS3 -> /CAN_RX
- U1 pad 2: /GPS_TX -> /SBUS
- U1 pad 20: /SBUS -> /CAN_TX
- U1 pad 21: unconnected-(U1-29_TX7-Pad21) -> /PICO_A_TX
- U1 pad 22: unconnected-(U1-30_CRX3-Pad22) -> /PICO_A_RX
- U1 pad 23: unconnected-(U1-31_CTX3-Pad23) -> GND
- U1 pad 24: /STEP_SLEEP -> unconnected-(U1-GPIO18-Pad24)
- U1 pad 25: /PWR_GOOD -> unconnected-(U1-GPIO19-Pad25)
- U1 pad 26: /TETHER_RX -> /LINK_A2B
- U1 pad 27: /TETHER_TX -> /LINK_B2A
- U1 pad 28: /WINCH_KILL -> GND
- U1 pad 29: /TETHER_DE -> /LEAK_EXC
- U1 pad 3: /GPS_RX -> GND
- U1 pad 30: unconnected-(U1-38_CS1_IN1-Pad30) -> /PICO_A_RUN
- U1 pad 31: /LEAK_EXC -> /S12_ADC
- U1 pad 33: /LEAK_R -> GND
- U1 pad 34: GND -> /LEAK_R
- U1 pad 36: unconnected-(U1-14_A0_TX3_SPDIF_OUT-Pad36) -> +3V3
- U1 pad 38: unconnected-(U1-16_A2_RX4_SCL1-Pad38) -> GND
- U1 pad 39: /S12_ADC -> /PICO_A_VSYS
- U1 pad 4: unconnected-(U1-2_OUT2-Pad4) -> /STEP_DIR
- U1 pad 40: /I2C_SDA -> unconnected-(U1-VBUS-Pad40)
- U1 pad 5: unconnected-(U1-3_LRCLK2-Pad5) -> /STEP
- U1 pad 6: /WINCH_PWM -> /STEP_SLEEP
- U1 pad 7: /LED_DIN -> /STEP_MS3
- U1 pad 8: /STEP -> GND
- U1 pad 9: /STEP_DIR -> /STEP_MS2
Routing:
- net /PICO_A_RUN: track 0.00 -> 93.6 mm, vias 0 -> 1
- net /+VELEC: track 274.9 -> 190.1 mm, vias 8 -> 2
- net /STEP_MS1: track 163.9 -> 88.5 mm, vias 1 -> 0
- net /SBUS: track 121.1 -> 47.3 mm, vias 2 -> 0
- net +5V: track 100.8 -> 27.3 mm, vias 3 -> 5
- net /STEP_MS3: track 158.3 -> 86.1 mm, vias 1 -> 0
- net /STEP_MS2: track 160.5 -> 92.4 mm
- net /LEAK_L: track 129.5 -> 63.7 mm, vias 2 -> 1
- net /CH5_SDA: track 122.0 -> 58.5 mm
- net /LEAK_R: track 107.4 -> 44.0 mm, vias 2 -> 0
- net /WINCH_KILL: track 122.9 -> 63.1 mm, vias 1 -> 0
- net +3V3: track 125.9 -> 67.4 mm, vias 8 -> 6
- net /STEP_EN: track 171.7 -> 113.8 mm, vias 1 -> 2
- net /PICO_B_RUN: track 0.00 -> 57.7 mm
- net /STEP_SLEEP: track 137.4 -> 81.4 mm, vias 1 -> 0
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Other:
- board text added: "PICO A CONTROL"
- board text added: "PICO B SENSORS"
- board text added: "RESET A"
- board text added: "RESET B"
- board text added: "USB (OPTIONAL)"
- board text added: "rev E 2026-10-13"
- board text removed: "CUT TEENSY VIN-VUSB BEFORE FITTING"
- board text removed: "rev D 2026-09-28"

Commit message: chore(pcb): V3 carrier and pod order-number markers for PCBWay
Like V3.1, the V3 carrier and the pod will be made by PCBWay, so their
back-silk order-number markers change from JLCPCB's "JLCJLCJLCJLC" to
PCBWay's "WayWayWay" (same spot, size and angle). Pick "Specify a
location" for the product number at checkout. Silkscreen only: the back
silkscreen gerber is the only one that changes on each board. CLAUDE.md
gets a short note on ordering.

Boat_PCB_V3 (rev E): 130.6 x 101.5 mm, 137 footprints, unchanged.
Pod_PCB_V3 (rev B): 48 x 63 mm, 54 footprints, unchanged.
Both: DRC 0 -> 0, unconnected 0 -> 0, schematic parity 0 -> 0, ERC 0 -> 0.
Boat_PCB_V3_1 stays at 0 on all four.

Co-Authored-By: Claude Opus 5.5 <noreply@anthropic.com>
Other:
- board text added: "WayWayWay"
- board text removed: "JLCJLCJLCJLC"
Changed lines of the file:
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@@
 		)
 	)
-	(gr_text "JLCJLCJLCJLC"
+	(gr_text "WayWayWay"
 		(at 59.499327 57.806412 0)
 		(layer "B.SilkS")
