File: Boat_PCB/Boat_PCB_V3/Boat_PCB_V3.kicad_sch (KiCad schematic)
At the start: 96 parts, among them J1 GPS M10-25Q, J10 Winch ESC, J11 12S HV tap, J12 Raspberry Pi 5 GPIO, J13 XT60 M18 ELECTRONICS, J14 XT60 M18 WINCH, J15 Drive shunt sense (off-board), J16 XT60 WINCH ESC OUT, J2 Pod tether, J3 CAN stub to VESCs, J4 SHT45 external, J5 Radar stepper motor, J6 Status LED, J7 SBUS RC receiver, J8 Hull leak left, J9 Hull leak right, Q1 P-FET 40V Rds<=10m, Q2 BSS138, U1 Teensy4.1, U10 INA228 electronics, U11 INA228 winch, U12 XIAO_ESP32_S3, U2 TCA9548A I2C mux, U3 TJA1051T/3 CAN xcvr, U4 BNO085, U5 ADXL375, U6 BMP390 breakout, U7 BH1750FVI-TR, U8 SHT45 internal, U9 INA228 drive

Commit message: feat(pcb): 12S drive rail is voltage-only; drop the drive shunt chain
Drive pack is 12S LiPo (2x 6S in series) = 50.4 V max, not the 63 V that
V3_PCB_SESSION_CONTEXT.md states and not M18 as README.md says. Corrections
recorded in docs/v3/v3_review_2026-08-05.md rather than editing the verbatim
planning files.

Decision: no current sensing on the 12S rail, just the ADC voltage tap. An
INA228 with nothing across Vin+/Vin- measures nothing, so the whole chain goes:
U9, C19, J15, R1, R2, R13, C7, plus the +VDRIVE / DRIVE_SENSE / DRIVE_ADC /
SH_DRIVE_P / SH_DRIVE_N nets and the off-board 250 uOhm shunt with its 4-wire
harness. 96 -> 89 components, and Teensy A2 frees up.

That also settles the J11/J15 redundancy: both were reading the same rail
through identical 220k/13k dividers. The 12S rail now has one sense path,
J11 -> 12S_RAW -> R7/R8 -> S12_SENSE -> R14 -> S12_ADC -> Teensy A3, giving
2.81 V at 50.4 V with 15 % headroom.

Drive current telemetry is not lost - the VESCs report per-motor current over
CAN, which distinguishes the two motors where a pack total would not. What goes
is the independent board-level cross-check against the ~90 A pack limit.

Fixed en route: the drive divider was 56k/10k, carried over from the V2 bench
where drive is 2x M18 in parallel at 21 V. On a 50.4 V rail that lands 9.55 V on
a 3.3 V ADC pin. Corrected to 220k/13k before the chain was removed entirely.

Also decided: leak auto-retract takes priority over the winch kill. The kill is
software-controlled, so this is a firmware precedence rule - assert the kill only
after retraction completes, and never latch it in a way that blocks retract.

Reference designators deliberately not renumbered; gaps at C3, C7, C19, R1, R2,
R13, U9, J15. Renumbering means rewriting every entry in the wiring table and a
slip there is a silent mis-wire. Conn_DriveSense_1x04 stays in the library,
now unused.

Verification: five passes clean - netlist/PDF/symbol/footprint exports load, all
89 components have fo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
Parts:
- removed C19, C7: 100nF, dreams_v3:C_Disc_D5.0mm_W2.5mm_P5.00mm, symbol dreams_v3:C
- removed J15: Drive shunt sense (off-board), dreams_v3:JST_XH_B4B-XH-A_1x04_P2.50mm_Vertical, symbol dreams_v3:Conn_DriveSense_1x04
- removed R1: 56k, dreams_v3:R_Axial_DIN0207_L6.3mm_D2.5mm_P10.16mm_Horizontal, symbol dreams_v3:R
- removed R13: 1k, dreams_v3:R_Axial_DIN0207_L6.3mm_D2.5mm_P10.16mm_Horizontal, symbol dreams_v3:R
- removed R2: 10k, dreams_v3:R_Axial_DIN0207_L6.3mm_D2.5mm_P10.16mm_Horizontal, symbol dreams_v3:R
- removed U9: INA228 drive, dreams_v3:HVSSOP-10-1EP_3x3mm_P0.5mm_EP1.83x1.89mm, symbol dreams_v3:INA228
Connections:
- net DRIVE_ADC: no longer names the net of U1.38 (16_A2_RX4_SCL1)
Other:
- note added: "BATTERY SENSE - 12S LiPo tap 220k/13k = 17.9x (50.4V), elec + winch 56k/10k = 6.6x (21V), plus a 1k series into each ADC pin. R1/R2/R13 removed with the drive shunt: the 12S rail is voltage-only now, on J11."
- note added: "CARRIER - CURRENT SENSE (M18 domains only; the 12S drive rail is voltage-only, and the VESCs already report per-motor current over CAN)"
- note removed: "BATTERY SENSE - 56k/10k = 6.6x per M18 rail, 220k/13k = 17.9x on the 12S tap, plus a 1k series resistor from each tap into its ADC pin"
- note removed: "CARRIER - CURRENT SENSE (one per isolated M18 domain)"

Commit message: feat(pcb): V3 schematic - audit fixes, pod off-board, 5V fusing, passives
Schematic work from review-log updates 9-11, previously uncommitted.

Update 9 - independent five-pass audit, four blockers found and fixed:
BNO085 was strapped for a crystal that was never fitted; the winch kill
shared a UART with SBUS, and the shared pin defeated the fail-safe; the
pod schottky was fitted backwards; the XIAO's 3V3 regulator output was
tied to the carrier's +3V3. Seven pins had no defined state while the
Teensy is high-Z.

Update 10 - the pod becomes a separate board, and every 5 V branch that
leaves the carrier is fused: F1/F3 0.75 A and F2 1.25 A hold, one PTC per
external harness, so a flooded pod cannot brown out the Pi.

Update 11 - passive review. R3/R5 56k -> 68k (the elec/winch dividers hit
3.46 V worst-case against a 3.3 V ADC); four series resistors added on
nets that leave the board; three parts dropped; BOM 28 -> 20 lines.

Adds the five project footprints the board already referenced but that
were never committed: Crystal_SMD_3215, two Bel Fuse 0ZRE bodies,
MSOP-10 and MountingHole_3.2mm_M3. Without them a fresh clone opens the
board (footprints are embedded) but cannot re-sync it against the library.

Co-Authored-By: Claude Opus 5 <noreply@anthropic.com>
Parts:
- removed C23: 10uF 16V +5V bulk, dreams_v3:CP_Radial_D10.0mm_P5.00mm, symbol dreams_v3:C_Polarized
- removed C27: 100nF, dreams_v3:C_Disc_D5.0mm_W2.5mm_P5.00mm, symbol dreams_v3:C
- removed R37: 1k Q2 gate, dreams_v3:R_Axial_DIN0207_L6.3mm_D2.5mm_P10.16mm_Horizontal, symbol dreams_v3:R
- removed U12: XIAO_ESP32_S3, dreams_v3:MODULE_XIAO_ESP32_S3, symbol dreams_v3:XIAO_ESP32_S3
- added C28, C29: 22pF 50V C0G, dreams_v3:C_Disc_D3.0mm_W1.6mm_P2.50mm, symbol dreams_v3:C
- added C30: 470uF 35V, dreams_v3:CP_Radial_D10.0mm_P5.00mm, symbol dreams_v3:C_Polarized
- added C31: 100nF 50V X7R, dreams_v3:C_Disc_D5.0mm_W2.5mm_P5.00mm, symbol dreams_v3:C
- added F1, F3: PTC 0.75A hold, dreams_v3:Fuse_BelFuse_0ZRE0075FF_L11.5mm_W4.8mm, symbol dreams_v3:Polyfuse
- added F2: PTC 1.25A hold, dreams_v3:Fuse_BelFuse_0ZRE0125FF_L21.2mm_W5.3mm, symbol dreams_v3:Polyfuse
- added MH1, MH2, MH3, MH4: MountingHole, dreams_v3:MountingHole_3.2mm_M3, symbol dreams_v3:MountingHole
- added R38, R39, R40, R41, R42, R43, R44: 10k 1%, dreams_v3:R_Axial_DIN0207_L6.3mm_D2.5mm_P10.16mm_Horizontal, symbol dreams_v3:R
- added R45: 330R 1%, dreams_v3:R_Axial_DIN0207_L6.3mm_D2.5mm_P10.16mm_Horizontal, symbol dreams_v3:R
- added R46, R47, R48: 1k 1%, dreams_v3:R_Axial_DIN0207_L6.3mm_D2.5mm_P10.16mm_Horizontal, symbol dreams_v3:R
- added Y1: 32.768kHz CL=12.5pF 50ppm, dreams_v3:Crystal_SMD_3215-2Pin_3.2x1.5mm, symbol dreams_v3:Crystal
- C1: value 470uF 35V elec -> 470uF 35V
- C10, C11, C12, C13, C14, C15, C16, C17, C18, C20, C21, C22, C4, C5, C6, C8, C9: value 100nF -> 100nF 50V X7R
- C2: value 470uF 35V winch -> 470uF 35V
- C24: value 10uF 16V +3V3 bulk -> 10uF 25V
- C25: value 100uF 35V VMOT bulk -> 100uF 35V
- C26: value 470uF 35V winch out -> 470uF 35V
- R10, R15, R16, R17, R18, R19, R20, R21, R22, R23, R24, R25, R26, R27, R28, R29, R30, R31, R9: value 4.7k -> 4.7k 1%
- R11, R12, R14: value 1k -> 1k 1%
- R3, R5: value 56k -> 68k 1%
- R32: value 10m 1% elec shunt -> 10mR 1%
- R33: value 2m 1% winch shunt -> 2mR 1%
- R34: value 10k gate pull-up -> 10k 1%
- R35: value 10k gate drive -> 10k 1%
- R36: value 10k Q2 pull-down -> 10k 1%
- R4, R6: value 10k -> 10k 1%
- R7: value 220k -> 220k 1%
- R8: value 13k -> 13k 1%
- U10, U11: footprint dreams_v3:HVSSOP-10-1EP_3x3mm_P0.5mm_EP1.83x1.89mm -> dreams_v3:MSOP-10_3x3mm_P0.5mm
Connections:
- net +3V3: now also R38.1, R39.1, R40.1, R41.1, R42.1, R43.1, R44.1
- net +5V: now also C30.1, C31.1, F1.1, F2.1, F3.1; no longer D1.1 (K), J2.2 (5V), J6.2 (5V), J7.2 (5V)
- net GND: now also C28.2, C29.2, C30.2, C31.2
- net IMU_RST: now also R39.2
- net LEAK_L: now also R46.1; no longer J8.2 (LEAK)
- net LEAK_R: now also R47.1; no longer J9.2 (LEAK)
- net LED_DIN: now also R45.1; no longer J6.3 (DIN)
- net MUX_RST: now also R38.2
- net POD_5V: now also D1.1 (K), J2.2 (5V); no longer D1.2 (A)
- net PWR_GOOD: now also R42.2
- net SBUS: now also R48.1; no longer J7.3 (SBUS)
- net STEP_EN: now also R40.2
- net STEP_SLEEP: now also R41.2
- net WINCH_KILL: now also U1.28 (36_CS)
- net ENV_SCL: now reaches U4.15 (ENV_SCL)
- net ENV_SCL: now also R43.2
- net ENV_SDA: now reaches U4.16 (ENV_SDA)
- net ENV_SDA: now also R44.2
- net IMU_XOUT: now reaches U4.26 (XOUT32/CLKSEL1)
- net IMU_XOUT: now also C29.1, Y1.2
- net IMU_XIN: now reaches U4.27 (XIN32)
- net IMU_XIN: now also C28.1, Y1.1
- net WINCH_KILL_MCU: no longer names the net of U1.21 (29_TX7)
- new net LEAK_L_EXT: J8.2 (LEAK), R46.2
- new net LEAK_R_EXT: J9.2 (LEAK), R47.2
- new net LED_5V: F2.2, J6.2 (5V)
- new net LED_DIN_EXT: J6.3 (DIN), R45.2
- new net POD_5V_F: D1.2 (A), F1.2
- new net SBUS_5V: F3.2, J7.2 (5V)
- new net SBUS_EXT: J7.3 (SBUS), R48.2

Commit message: feat(pcb): carrier rev D and pod board rev A
Carrier (Boat_PCB/Boat_PCB_V3), against the pre-relayout board at c4b673b:

- Re-placed and re-routed for a Pi 5 mounted face down on 30 mm
  standoffs, fully inside the outline. The board goes from 132.0 x 108.4
  to 130.6 x 101.5 mm, 7 % less area.
- Review fixes. The A2 footprint was redrawn from Pololu's drill guide:
  the old one reversed the buck's pinout end for end. XT60 pin 1 is now
  negative, J16 is an XT60-F, J11 is a JST-VH, and the Kelvin sense taps
  have their own nets. Added: TVS D3/D4/D5, gate zener D2, power and winch
  LEDs, the U12 level shifter for the WS2812, the JP1 CAN termination
  option, series resistors on off-board nets, and TP1-TP6.
- Pod tether: pack voltage through F1 (0.40 A PTC), RS-485 through U13
  (THVD2410) with R62 and R63.
- Every resistor lies flat on the 10.16 mm footprint. The edge connectors
  share one row, and the resistors sit in aligned banks.
- Parts review: the electronics and winch 68k/10k ADC dividers, with their
  1k series resistors and filter caps, only duplicated the INA228 VBUS
  readings, so they came out. R14, C8 and C10 served no purpose. That is
  11 parts removed. Teensy pins 14 and 15 are free, and the 12S tap is now
  net S12_ADC.
- ERC 70 -> 0. DRC 107 -> 0 (60 silk overlaps, 29 under-width power
  tracks, 18 silk over copper). Schematic parity 154 -> 0. Unconnected
  0 -> 0. Footprints 108 -> 126.

Pod (Boat_PCB/Pod_PCB_V3), new: schematic and a 48 x 63 mm rev A layout,
with wire-solder pads instead of connectors. ERC 0, DRC 0, parity 0.

Library: footprints and symbols for both boards, 51 footprints in all.
The A2 and Pi-socket footprints were fixed so the board copies match the
library.

Docs: CLAUDE.md baselines, the design brief, both READMEs, and the
planning docs' scope notes.

Co-Authored-By: Claude Opus 5.5 <noreply@anthropic.com>
Parts:
- removed C10, C5, C6, C8: 100nF 50V X7R, dreams_v3:C_Disc_D5.0mm_W2.5mm_P5.00mm, symbol dreams_v3:C
- removed D1: Schottky pod 5V, dreams_v3:D_SOD-123, symbol dreams_v3:D_Schottky
- removed R11, R12, R14: 1k 1%, dreams_v3:R_Axial_DIN0207_L6.3mm_D2.5mm_P10.16mm_Horizontal, symbol dreams_v3:R
- removed R19, R20: 4.7k 1%, dreams_v3:R_Axial_DIN0207_L6.3mm_D2.5mm_P10.16mm_Horizontal, symbol dreams_v3:R
- removed R3, R5: 68k 1%, dreams_v3:R_Axial_DIN0207_L6.3mm_D2.5mm_P10.16mm_Horizontal, symbol dreams_v3:R
- removed R4, R41, R6: 10k 1%, dreams_v3:R_Axial_DIN0207_L6.3mm_D2.5mm_P10.16mm_Horizontal, symbol dreams_v3:R
- added C32, C34: 100nF 50V X7R, dreams_v3:C_Disc_D5.0mm_W2.5mm_P5.00mm, symbol dreams_v3:C
- added C33: 1uF 50V X7R, dreams_v3:C_Disc_D5.0mm_W2.5mm_P5.00mm, symbol dreams_v3:C
- added D2: 1N5245B 15V, dreams_v3:D_DO-35_SOD27_P7.62mm_Horizontal, symbol dreams_v3:D_Zener
- added D3, D4: SMBJ24A, dreams_v3:D_SMB, symbol dreams_v3:D_Zener
- added D5: SMBJ5.0A, dreams_v3:D_SMB, symbol dreams_v3:D_Zener
- added D6: NUP2105L, dreams_v3:SOT-23, symbol dreams_v3:NUP2105L
- added D7: green +5V, dreams_v3:LED_D3.0mm, symbol dreams_v3:LED
- added D8: green +3V3, dreams_v3:LED_D3.0mm, symbol dreams_v3:LED
- added D9: red WINCH ON, dreams_v3:LED_D3.0mm, symbol dreams_v3:LED
- added JP1: CAN TERM, dreams_v3:PinHeader_1x02_P2.54mm_Vertical, symbol dreams_v3:Jumper_2_Open
- added R49, R50, R53: 1k 1%, dreams_v3:R_Axial_DIN0207_L6.3mm_D2.5mm_P10.16mm_Horizontal, symbol dreams_v3:R
- added R54, R56, R57: 100k 1%, dreams_v3:R_Axial_DIN0207_L6.3mm_D2.5mm_P10.16mm_Horizontal, symbol dreams_v3:R
- added R55, R60, R62: 10k 1%, dreams_v3:R_Axial_DIN0207_L6.3mm_D2.5mm_P10.16mm_Horizontal, symbol dreams_v3:R
- added R58: 1.5k 1%, dreams_v3:R_Axial_DIN0207_L6.3mm_D2.5mm_P10.16mm_Horizontal, symbol dreams_v3:R
- added R59: 680R 1%, dreams_v3:R_Axial_DIN0207_L6.3mm_D2.5mm_P10.16mm_Horizontal, symbol dreams_v3:R
- added R61, R63: 120R 1%, dreams_v3:R_Axial_DIN0207_L6.3mm_D2.5mm_P10.16mm_Horizontal, symbol dreams_v3:R
- added TP1, TP2: GND, dreams_v3:TestPoint_Keystone_5000-5004_Miniature, symbol dreams_v3:TestPoint
- added TP3: +5V, dreams_v3:TestPoint_Keystone_5000-5004_Miniature, symbol dreams_v3:TestPoint
- added TP4: +3V3, dreams_v3:TestPoint_Keystone_5000-5004_Miniature, symbol dreams_v3:TestPoint
- added TP5: SDA, dreams_v3:TestPoint_Keystone_5000-5004_Miniature, symbol dreams_v3:TestPoint
- added TP6: SCL, dreams_v3:TestPoint_Keystone_5000-5004_Miniature, symbol dreams_v3:TestPoint
- added U12: 74AHCT1G125, dreams_v3:SOT-23-5, symbol dreams_v3:74AHCT1G125
- added U13: THVD2410, dreams_v3:SOIC-8_3.9x4.9mm_P1.27mm, symbol dreams_v3:THVD2410D
- C24: value 10uF 25V -> 10uF 25V X7R; footprint dreams_v3:CP_Radial_D10.0mm_P5.00mm -> dreams_v3:C_Disc_D5.0mm_W2.5mm_P5.00mm; symbol dreams_v3:C_Polarized -> dreams_v3:C
- C30: value 470uF 35V -> 470uF 16V low-ESR 105C; footprint dreams_v3:CP_Radial_D10.0mm_P5.00mm -> dreams_v3:CP_Radial_D8.0mm_P3.50mm
- F1: value PTC 0.75A hold -> PTC 0.40A hold
- J11: value 12S HV tap -> 12S HV tap (JST-VH); footprint dreams_v3:JST_XH_B2B-XH-A_1x02_P2.50mm_Vertical -> dreams_v3:JST_VH_B2P-VH_1x02_P3.96mm_Vertical
- J16: value XT60 WINCH ESC OUT -> XT60-F WINCH ESC OUT (female); footprint dreams_v3:AMASS_XT60-M_1x02_P7.20mm_Vertical -> dreams_v3:AMASS_XT60-F_1x02_P7.20mm_Vertical
- MH1, MH2, MH3, MH4: now left out of the parts list
- Q1: value P-FET 40V Rds<=10m -> IPP120P04P4L-03
Connections:
- net POD_5V_F is gone; now on net POD_VPACK: F1.2
- net S12_SENSE is gone; now on net S12_ADC: R7.2, R8.1
- net +3V3: now also C33.1, C34.1, R55.1, R59.1, TP4.1, U13.8 (VCC); no longer U4.4 (~{BOOT})
- net +5V: now also C32.1, D5.1 (K), R58.1, TP3.1, U12.5 (VCC); no longer F1.1
- net +VELEC: now also F1.1, D3.1 (K); no longer R32.3, U10.8 (Vbus), U10.9 (Vin-)
- net +VWINCH: now also D2.1 (K); no longer R33.3, U11.8 (Vbus), U11.9 (Vin-)
- net CANH: now also R61.1
- net CANL: now also JP1.2 (B)
- net GND: now also J13.1 (-), J14.1 (-), J16.1 (-), C32.2, C33.2, C34.2, D3.2 (A), D4.2 (A), D5.2 (A), D6.3 (A), D7.1 (K), D8.1 (K), D9.1 (K), R54.2, R62.2, TP1.1, TP2.1, U12.1, U12.3 (GND), U13.5 (GND); no longer J13.2 (-), J14.2 (-), J16.2 (-), U7.2 (ADDR)
- net GPS_RX: now also R50.1; no longer J1.2 (RX)
- net GPS_TX: now also R49.2; no longer J1.1 (TX)
- net I2C_SCL: now also TP6.1
- net I2C_SDA: now also TP5.1
- net LEAK_L: now also U1.32 (40_A16), R56.2; no longer U1.4 (2_OUT2)
- net LEAK_R: now also U1.33 (41_A17), R57.2; no longer U1.5 (3_LRCLK2)
- net LED_DIN: now also U12.2; no longer R45.1
- net SH_ELEC_P: now also J13.2 (+); no longer J13.1 (+), R32.2, U10.10 (Vin+)
- net SH_WINCH_P: now also J14.2 (+); no longer J14.1 (+), R33.2, U11.10 (Vin+)
- net TETHER_A: now also D6.1 (K), R63.1, U13.6 (A); no longer U1.27 (35_TX8)
- net TETHER_B: now also D6.2 (K), R63.2, U13.7 (B); no longer U1.26 (34_RX8)
- net WINCH_GATE: now also D2.2 (A)
- net WINCH_PWM: now also R53.1; no longer J10.2 (PWM)
- net WINCH_SW: now also J16.2 (+), D4.1 (K), R60.1; no longer J16.1 (+)
- net TETHER_DE: now reaches U1.29 (37_CS)
- net TETHER_DE: now also R62.1, U13.2 (~{RE}), U13.3 (DE)
- net LEAK_EXC: now reaches U1.31 (39_MISO1_OUT1A)
- net LEAK_EXC: now also R56.1, R57.1
- net ELEC_ADC: no longer names the net of U1.36 (14_A0_TX3_SPDIF_OUT)
- net POD_5V renamed POD_VPACK
- net WINCH_ADC: no longer names the net of U1.37 (15_A1_RX3_SPDIF_IN)
- new net BH_ADDR: R54.1, U7.2 (ADDR)
- new net CAN_TERM: JP1.1 (A), R61.2
- new net ELEC_SHUNT_N: R32.3, U10.8 (Vbus), U10.9 (Vin-)
- new net ELEC_SHUNT_P: R32.2, U10.10 (Vin+)
- new net GPS_RX_EXT: J1.2 (RX), R50.2
- new net GPS_TX_EXT: J1.1 (TX), R49.1
- new net IMU_BOOTN: R55.2, U4.4 (~{BOOT})
- new net LED_DIN_5V: R45.1, U12.4
- new net LED_P3V3: D8.2 (A), R59.2
- new net LED_P5V: D7.2 (A), R58.2
- new net LED_WINCH: D9.2 (A), R60.2
- new net TETHER_RX: U1.26 (34_RX8), U13.1 (RO)
- new net TETHER_TX: U1.27 (35_TX8), U13.4 (DI)
- new net WINCH_PWM_EXT: J10.2 (PWM), R53.2
- new net WINCH_SHUNT_N: R33.3, U11.8 (Vbus), U11.9 (Vin-)
- new net WINCH_SHUNT_P: R33.2, U11.10 (Vin+)
- no-connect marks 0 -> 58
Other:
- note added: "BATTERY SENSE - 12S LiPo tap 220k/13k = 17.9x (50.4V), elec + winch 68k/10k = 7.8x (2.69 V at 21 V), plus a 1k series into each ADC pin. R1/R2/R13 removed with the drive shunt: the 12S rail is voltage-only now, on J11."
- note added: "BRING-UP - test points, power LEDs, WINCH ON LED, optional CAN termination (fit JP1 only if this node ends the bus)"
- note added: "CAPACITORS - 470uF bulk per M18 pack; 100nF ADC filters (V2 had none). The 12S tap filter cap is C4 at the Teensy pin; J11 is JST-VH so no signal plug can mate with it."
- note added: "CONNECTORS - JST-XH for signals, JST-VH for the 12S tap, XT60 for packs; J16 is female (switched output)"
- note added: "HULL LEAK - probes on ADC pins 40/41, excited from pin 39 only while sampling (reads fresh water, limits probe electrolysis)"
- note added: "I2C PULL-UPS - 4.7k pair on every used TCA9548A channel except CH2, where the BMP390 breakout (U6) has its own (a mux isolates the channels, so the upstream pair does not serve them)"
- note added: "M18 PACK INPUTS - XT60 (pin 1 = notched end = negative, per the XT60 convention) + in-line Kelvin shunts; the sense pins have their own nets (ELEC/WINCH_SHUNT_P/N). Drive is sensed off-board: its pack never reaches this carrier."
- note added: "POD PCB - separate board, here for reference only. Tether pin 2 carries the electronics pack voltage (M18, 15-21 V) through F1; the pod makes its own 5 V."
- note added: "PROTECTION - TVS on both pack rails (also a reverse-polarity crowbar that blows the pack fuse), +5V over-voltage clamp, Q1 gate clamp, tether TVS (24 V NUP2105L, D6)"
- note added: "REV C ADDITIONS (2026-09-24 review) - every part here connects through net labels"
- note added: "SERIES RESISTORS ON EVERY OFF-BOARD SIGNAL (brief rule) - GPS UART and winch ESC PWM. The pod tether is RS-485 now (U13, see TETHER RS-485), which needs none"
- note added: "TETHER RS-485 (2026-09-25) - half duplex on Serial8 (TX8 pin 35, RX8 pin 34); pin 37 drives DE and ~RE together (Serial8.transmitterEnable(37)); R62 holds receive mode through reset; 120R termination at this end of the tether. RX idles high on the Teensy RX pull-up while transmitting."
- note added: "WS2812 LEVEL SHIFT (3.3 V Teensy -> 5 V LED data) + SENSOR STRAPS"
- note removed: "BATTERY SENSE - 12S LiPo tap 220k/13k = 17.9x (50.4V), elec + winch 56k/10k = 6.6x (21V), plus a 1k series into each ADC pin. R1/R2/R13 removed with the drive shunt: the 12S rail is voltage-only now, on J11."
- note removed: "CAPACITORS - 470uF bulk per M18 pack; 100nF ADC filters (V2 had none). The 12S tap cap is fitted off-board on the wiring, so there is no C3 here."
- note removed: "CONNECTORS - all JST-XH, pins named per function"
- note removed: "I2C PULL-UPS - 4.7k pair on every used TCA9548A channel (a mux isolates them, so the upstream pair does not serve the channels)"
- note removed: "M18 PACK INPUTS - XT60 + in-line Kelvin shunts. Drive is sensed off-board: its pack never reaches this carrier."
- note removed: "POD PCB - separate board, here for reference only"
