File: Boat_PCB/Boat_PCB_V3/Boat_PCB_V3.kicad_sch (KiCad schematic)
At the start: 126 parts, among them J1 GPS M10-25Q, J10 Winch ESC, J11 12S HV tap (JST-VH), J12 Raspberry Pi 5 GPIO, J13 XT60 M18 ELECTRONICS, J14 XT60 M18 WINCH, J16 XT60-F WINCH ESC OUT (female), J2 Pod tether, J3 CAN stub to VESCs, J4 SHT45 external, J5 Radar stepper motor, J6 Status LED, J7 SBUS RC receiver, J8 Hull leak left, J9 Hull leak right, Q1 IPP120P04P4L-03, Q2 BSS138, U1 Teensy4.1, U10 INA228 electronics, U11 INA228 winch, U12 74AHCT1G125, U13 THVD2410, U2 TCA9548A I2C mux, U3 TJA1051T/3 CAN xcvr, U4 BNO085, U5 ADXL375, U6 BMP390 breakout, U7 BH1750FVI-TR, U8 SHT45 internal, Y1 32.768kHz CL=12.5pF 50ppm

Commit message: feat(pcb): V3 carrier rev E: two Pico 2s, Pi link on the header
Rev E replaces the Teensy 4.1 with two Raspberry Pi Pico 2s, one job each,
after V3.1 tried one Pico: Pico A (U1) runs control (CAN on can2040, SBUS,
winch, stepper, LED, leak sensing, 12S ADC) and Pico B (U14) the sensors
(I2C mux, GPS, pod RS-485), joined by a UART link. Both are socketed under
the carrier, take VSYS from +5V through D10/D11 and have reset buttons
SW1/SW2. R36/R62 drop to 4.7k for RP2350 erratum E9.

The Pi talks to Pico A over its GPIO header instead of USB, so its USB
ports stay free for cameras and the modem: Pi UART0 (GPIO14/15) runs to
Pico A GP17/GP16 through 1k series resistors (R66/R67), so neither end can
back-power the other, and GPIO23/24 reset Pico A/B through BSS138s (Q3/Q4)
across SW1/SW2, held off by 100k pull-downs (R64/R65). The Picos' USB stays
usable: VBUS isn't wired on the carrier.

C25 (A4988 VMOT bulk) goes from 100 uF to 470 uF 35 V, so C1, C2, C25 and
C26 all take the Rubycon caps already on hand (listed in the parts doc).

Library: RaspberryPi_Pico pin 3 (GND) is power_in now, since two Picos on
one GND net were a power-output conflict; the V3.1 schematic gets a GND
PWR_FLAG to match.

Boat_PCB_V3, rev D -> rev E: 126 -> 137 footprints, 5356 -> 4198 mm of
track, 142 -> 118 vias. DRC 0 -> 0, unconnected 0 -> 0, schematic parity
0 -> 0, ERC 0 -> 0. Boat_PCB_V3_1 and Pod_PCB_V3: DRC, parity and ERC stay
at 0.

Docs: CLAUDE.md pin maps and hardware facts, README, design brief, V3 docs
index, V3.1 doc, session context, parts doc and lib README; this week's
update bullet.

Co-Authored-By: Claude Opus 5.5 <noreply@anthropic.com>
Parts:
- removed U1: Teensy4.1, dreams_v3:Teensy41, symbol dreams_v3:Teensy4.1
- added D10, D11: B5819W, dreams_v3:D_SOD-123, symbol dreams_v3:D_Schottky
- added Q3, Q4: BSS138, dreams_v3:SOT-23, symbol dreams_v3:Q_NMOS_GSD
- added R64, R65: 100k 1%, dreams_v3:R_Axial_DIN0207_L6.3mm_D2.5mm_P10.16mm_Horizontal, symbol dreams_v3:R
- added R66, R67: 1k 1%, dreams_v3:R_Axial_DIN0207_L6.3mm_D2.5mm_P2.54mm_Vertical, symbol dreams_v3:R
- added SW1: PICO A RESET, dreams_v3:SW_PUSH_6mm, symbol dreams_v3:SW_Push
- added SW2: PICO B RESET, dreams_v3:SW_PUSH_6mm, symbol dreams_v3:SW_Push
- added U1, U14: Raspberry Pi Pico 2, dreams_v3:RaspberryPi_Pico_Socketed_THT, symbol dreams_v3:RaspberryPi_Pico
- C25: value 100uF 35V -> 470uF 35V
- R36, R62: value 10k 1% -> 4.7k 1%
Connections:
- net +3V3: now also U1.36 (3V3)
- net +5V: now also D10.2 (A), D11.2 (A)
- net ADXL_INT1: now also U14.25 (GPIO19)
- net ADXL_INT2: now also U14.26 (GPIO20)
- net BMP_INT: now also U14.9 (GPIO6)
- net CAN_RX: now also U1.19 (GPIO14)
- net CAN_TX: now also U1.20 (GPIO15)
- net GND: now also Q3.2 (S), Q4.2 (S), R64.2, R65.2, SW1.1, SW2.1, U1.13 (GND), U1.18 (GND), U1.23 (GND), U1.28 (GND), U1.3 (GND), U1.33 (AGND), U1.38 (GND), U1.8 (GND), U14.13 (GND), U14.18 (GND), U14.23 (GND), U14.28 (GND), U14.3 (GND), U14.33 (AGND), U14.38 (GND), U14.8 (GND)
- net GPS_RX: now also U14.6 (GPIO4)
- net GPS_TX: now also U14.7 (GPIO5)
- net I2C_SCL: now also U14.17 (GPIO13)
- net I2C_SDA: now also U14.16 (GPIO12)
- net IMU_INT: now also U14.11 (GPIO8)
- net IMU_RST: now also U14.12 (GPIO9)
- net INA_ALERT: now also U14.10 (GPIO7)
- net LEAK_EXC: now also U1.29 (GPIO22)
- net LEAK_L: now also U1.32 (GPIO27_ADC1)
- net LEAK_R: now also U1.34 (GPIO28_ADC2)
- net LED_DIN: now also U1.14 (GPIO10)
- net MUX_RST: now also U14.19 (GPIO14)
- net PWR_GOOD: now also U1.15 (GPIO11)
- net S12_ADC: now also U1.31 (GPIO26_ADC0)
- net SBUS: now also U1.2 (GPIO1)
- net STEP: now also U1.5 (GPIO3)
- net STEP_DIR: now also U1.4 (GPIO2)
- net STEP_EN: now also U1.11 (GPIO8)
- net STEP_MS1: now also U1.10 (GPIO7)
- net STEP_MS2: now also U1.9 (GPIO6)
- net STEP_MS3: now also U1.7 (GPIO5)
- net STEP_SLEEP: now also U1.6 (GPIO4)
- net TETHER_DE: now also U14.24 (GPIO18)
- net TETHER_RX: now also U14.22 (GPIO17)
- net TETHER_TX: now also U14.21 (GPIO16)
- net WINCH_KILL: now also U1.12 (GPIO9)
- net WINCH_PWM: now also U1.1 (GPIO0)
- net PI_RX: now reaches J12.10 (GPIO15_RXD)
- net PI_RX: now also R67.1
- net PI_RST_A: now reaches J12.16 (GPIO23)
- net PI_RST_A: now also Q3.1 (G), R64.1
- net PI_RST_B: now reaches J12.18 (GPIO24)
- net PI_RST_B: now also Q4.1 (G), R65.1
- net PI_TX: now reaches J12.8 (GPIO14_TXD)
- net PI_TX: now also R66.1
- new net LINK_A2B: U1.26 (GPIO20), U14.15 (GPIO11)
- new net LINK_B2A: U1.27 (GPIO21), U14.14 (GPIO10)
- new net PICO_A_RUN: Q3.3 (D), SW1.2, U1.30 (RUN)
- new net PICO_A_RX: R66.2, U1.22 (GPIO17)
- new net PICO_A_TX: R67.2, U1.21 (GPIO16)
- new net PICO_A_VSYS: D10.1 (K), U1.39 (VSYS)
- new net PICO_B_RUN: Q4.3 (D), SW2.2, U14.30 (RUN)
- new net PICO_B_VSYS: D11.1 (K), U14.39 (VSYS)
- no-connect marks 58 -> 51
Other:
- note added: "CAPACITORS - 470uF bulk per M18 pack; 100nF ADC filters (V2 had none). The 12S tap filter cap is C4 at Pico A's ADC0 pin; J11 is JST-VH so no signal plug can mate with it."
- note added: "HULL LEAK - probes on Pico A's ADC1/ADC2 (GP27/GP28), excited from GP22 only while sampling (reads fresh water, limits probe electrolysis)"
- note added: "PI LINK (rev E, 2026-10-13)"
- note added: "Pi UART0 (GPIO14 TX / GPIO15 RX, header pins 8 / 10) to Pico A GP17 / GP16 (its UART0 RX / TX). R66 / R67 (1k) in those lines stop either end back-powering the other through its pin. Pico A's UART0 can't also take SBUS on GP1: run SBUS or this link on the PIO. Pi GPIO23 / GPIO24 (header pins 16 / 18) high resets Pico A / B through Q3 / Q4, across SW1 / SW2. R64 / R65 hold them off while the Pi is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"
- note added: "Pico A (U1, next to the Pi header): control. CAN on the PIO (can2040), SBUS, winch PWM + kill, stepper, WS2812, leak probes, 12S ADC. Pico B (U14, here): sensors. TCA9548A I2C mux, GPS, pod RS-485. A UART link joins them: LINK_A2B / LINK_B2A. Both sit socketed under the carrier, each with a USB cable to the Pi. VSYS from +5V through D10 / D11. Pico A's 3V3 pin is the board's +3V3 rail; Pico B's 3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"
- note added: "TETHER RS-485 (2026-09-25, Pico B since 2026-10-13) - half duplex on Pico B's UART0 (TX GP16, RX GP17); GP18 drives DE and ~RE together (high = transmit); R62 holds receive mode through reset; 120R termination at this end of the tether."
- note added: "TWO PICO 2s (replaced the Teensy 4.1, 2026-10-13)"
- note added: "WS2812 LEVEL SHIFT (3.3 V Pico A -> 5 V LED data) + SENSOR STRAPS"
- note removed: "CAPACITORS - 470uF bulk per M18 pack; 100nF ADC filters (V2 had none). The 12S tap filter cap is C4 at the Teensy pin; J11 is JST-VH so no signal plug can mate with it."
- note removed: "HULL LEAK - probes on ADC pins 40/41, excited from pin 39 only while sampling (reads fresh water, limits probe electrolysis)"
- note removed: "TETHER RS-485 (2026-09-25) - half duplex on Serial8 (TX8 pin 35, RX8 pin 34); pin 37 drives DE and ~RE together (Serial8.transmitterEnable(37)); R62 holds receive mode through reset; 120R termination at this end of the tether. RX idles high on the Teensy RX pull-up while transmitting."
- note removed: "WS2812 LEVEL SHIFT (3.3 V Teensy -> 5 V LED data) + SENSOR STRAPS"

Commit message: feat(pcb): V3 carrier rev F, 10S power
Kyle, 2026-10-14: the full V3 runs from two 10S 10 Ah Li-ion packs in parallel, one
bus (30-42 V) for the drives, J13 (electronics) and J14 (winch), with an optional 4S
backup for the 5 V side. Rev E's electronics and winch inputs were 15-21 V domains.

Rated for 42 V:
- D3/D4 SMBJ24A -> SMBJ43A, Q1 IPP120P04P4L-03 -> SUP90P06-09L (-60 V);
- C1/C2/C26 470 uF 35 V -> 100 uF 63 V, R60 10k -> 22k.
New parts:
- U15, a Pololu D36V6F15 on the underside: +15V for the A4988 (it tops out at 35 V)
  and, through F1 and the In2 run along the top edge, the pod tether;
- D12/D13 (B360B), a diode-OR of the 10S rail and the 4S backup into the 5 V buck A2;
- J18, the 4S backup input (JST-VH), on the underside with its plug from below.
Nets: 12S_RAW/S12_ADC -> PACK_RAW/PACK_ADC, POD_VPACK -> POD_15V; new +VLOGIC,
+VBACKUP, +15V. No part moved. A placement search found the only spots that clear
every courtyard and through-hole pad, and the power runs are hand-placed.

Carrier: footprints 137 -> 141; ERC 0 -> 0, DRC 0 -> 0, unconnected 0 -> 0,
parity 0 -> 0, no exclusions. V3.1 and the pod are unchanged (all 0).

Docs follow: CLAUDE.md (terms, safety rules, pack sensing), README, Boat_PCB/CLAUDE.md
(baseline, placement, locked copper), the brief, the docs index, V3_MECHANICAL 1.1,
the scope notes of both planning files, and this week's update bullet.

Co-Authored-By: Claude Opus 5.5 <noreply@anthropic.com>
Parts:
- added D12, D13: B360B, dreams_v3:D_SMB, symbol dreams_v3:D_Schottky
- added J18: 4S backup (JST-VH), dreams_v3:JST_VH_B2P-VH_1x02_P3.96mm_Vertical, symbol dreams_v3:Conn_12S_Tap_1x02
- added U15: Pololu D36V6F15 15V 600mA, dreams_v3:Pololu_D36V6F5, symbol dreams_v3:Pololu_D36V6F5
- C1, C2, C26: value 470uF 35V -> 100uF 63V
- D3, D4: value SMBJ24A -> SMBJ43A
- J11: value 12S HV tap (JST-VH) -> 10S pack tap (JST-VH)
- J13: value XT60 M18 ELECTRONICS -> XT60 10S ELECTRONICS
- J14: value XT60 M18 WINCH -> XT60 10S WINCH
- Q1: value IPP120P04P4L-03 -> SUP90P06-09L
- R60: value 10k 1% -> 22k 1%
Connections:
- net +VELEC: now also D12.2 (A), U15.2 (VIN); no longer A1.8 (VMOT), A2.7 (VIN), A2.8 (VIN), C25.1, F1.1
- net GND: now also J18.1 (GND), U15.3 (GND)
- net 12S_RAW renamed PACK_RAW
- net POD_VPACK renamed POD_15V
- net S12_ADC renamed PACK_ADC
- new net +15V: A1.8 (VMOT), C25.1, F1.1, U15.4 (VOUT)
- new net +VBACKUP: D13.2 (A), J18.2 (VIN)
- new net +VLOGIC: A2.7 (VIN), A2.8 (VIN), D12.1 (K), D13.1 (K)
- no-connect marks 51 -> 52
Other:
- note added: "10S INPUTS - XT60 (pin 1 = notched end = negative, per the XT60 convention) + in-line Kelvin shunts; the sense pins have their own nets (ELEC/WINCH_SHUNT_P/N). Both packs share one 10S bus; the drive is sensed off-board: its current never crosses this carrier."
- note added: "10S POWER (rev F, 2026-10-14)"
- note added: "BATTERY SENSE - 10S pack tap J11, 220k/13k = 17.9x (2.34 V at 42 V, room up to 12S), plus C4 at Pico A's ADC0. Electronics and winch voltages come from the INA228s (U10, U11)."
- note added: "CAPACITORS - 100uF 63V bulk on each 10S input; 470uF 35V on the 15 V A4988 supply (C25); 100nF ADC filters. The pack tap filter cap is C4 at Pico A's ADC0 pin; J11 is JST-VH so no signal plug can mate with it."
- note added: "CARRIER - CURRENT SENSE (electronics and winch feeds only; the drive is voltage-only, and the VESCs already report per-motor current over CAN)"
- note added: "CONNECTORS - JST-XH for signals, JST-VH for the 10S tap (J11) and the 4S backup (J18), XT60 for the 10S inputs; J16 is female (switched output)"
- note added: "POD PCB - separate board, here for reference only. Tether pin 2 carries 15 V from U15 through F1; the pod makes its own 5 V."
- note added: "PROTECTION - 43 V TVS on both 10S rails (also a reverse-polarity crowbar that blows the pack fuse), +5V over-voltage clamp, Q1 gate clamp, tether TVS (24 V NUP2105L, D6)"
- note added: "Two 10S 10 Ah Li-ion packs in parallel make one 10S bus (30-42 V): drives, J13 and J14. +VELEC (10S, after R32) feeds three things: the 5 V buck A2 through D12, diode-ORed with an optional 4S backup on J18 through D13 (+VLOGIC); U15, +15V for the A4988's motor supply (it tops out at 35 V) and, through F1, the pod tether, as on V3.1. 600 mA in all: the pod takes about 0.13 A, the stepper the rest.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"
- note removed: "BATTERY SENSE - 12S LiPo tap 220k/13k = 17.9x (50.4V), elec + winch 68k/10k = 7.8x (2.69 V at 21 V), plus a 1k series into each ADC pin. R1/R2/R13 removed with the drive shunt: the 12S rail is voltage-only now, on J11."
- note removed: "CAPACITORS - 470uF bulk per M18 pack; 100nF ADC filters (V2 had none). The 12S tap filter cap is C4 at Pico A's ADC0 pin; J11 is JST-VH so no signal plug can mate with it."
- note removed: "CARRIER - CURRENT SENSE (M18 domains only; the 12S drive rail is voltage-only, and the VESCs already report per-motor current over CAN)"
- note removed: "CONNECTORS - JST-XH for signals, JST-VH for the 12S tap, XT60 for packs; J16 is female (switched output)"
- note removed: "M18 PACK INPUTS - XT60 (pin 1 = notched end = negative, per the XT60 convention) + in-line Kelvin shunts; the sense pins have their own nets (ELEC/WINCH_SHUNT_P/N). Drive is sensed off-board: its pack never reaches this carrier."
- note removed: "POD PCB - separate board, here for reference only. Tether pin 2 carries the electronics pack voltage (M18, 15-21 V) through F1; the pod makes its own 5 V."
- note removed: "PROTECTION - TVS on both pack rails (also a reverse-polarity crowbar that blows the pack fuse), +5V over-voltage clamp, Q1 gate clamp, tether TVS (24 V NUP2105L, D6)"

Commit message: feat(pcb): carrier rev F without the BMP390, condensed to 130.6 x 95.5 mm
The BMP390 breakout (U6) came off with its tracks. Its one job, a surface baseline
for the pod's pressure depth, went when depth moved to the fish-finder sonar. Mux
CH2 and Pico B GP6 are free.

With U6's area free, the bottom edge came up 6 mm. J1 (GPS) and J4 (SHT45 external)
moved into U6's old spot, because the Pi's USB jacks hang over the bottom-right
corner. The bottom connector row, its resistors and A1 moved up. J18, SW1/SW2 and
MH3/MH4 moved, and the In2 +5V zone was re-shaped. Everything that touched a moved
part was re-routed.

Carrier (Boat_PCB_V3), before -> after:
- footprints 141 -> 140
- size 130.6 x 101.5 -> 130.6 x 95.5 mm
- ERC 0 -> 0, DRC 0 -> 0, unconnected 0 -> 0, schematic parity 0 -> 0

Re-routing took tracks from 4105 to 4439 mm and vias from 119 to 141.

Docs, this week's update and the site's board renders, 3D model, poster and
callouts follow the board.

Co-Authored-By: Claude Opus 5.5 <noreply@anthropic.com>
Parts:
- removed U6: BMP390 breakout, dreams_v3:BMP390, symbol dreams_v3:BMP390
Connections:
- net BMP_INT: no longer names the net of U14.9 (GPIO6)
- net CH2_SCL: no longer names the net of U2.9 (SC2)
- net CH2_SDA: no longer names the net of U2.8 (SD2)
- no-connect marks 52 -> 54
Other:
- note added: "I2C PULL-UPS - 4.7k pair on every used TCA9548A channel (a mux isolates the channels, so the upstream pair does not serve them). CH2 is free: the BMP390 (U6) came off in rev F"
- note removed: "I2C PULL-UPS - 4.7k pair on every used TCA9548A channel except CH2, where the BMP390 breakout (U6) has its own (a mux isolates the channels, so the upstream pair does not serve them)"
